File: PCB/TRIO Rp2040.kicad_sch (KiCad schematic)
At the start: 27 parts, among them J1 USB_C_Receptacle_USB2.0_16P, J2 Conn_01x02_Pin, J3 Conn_01x02_Pin, J5 Conn_01x07_Pin, J6 Conn_01x07_Pin, J7 Conn_01x07_Pin, SW1 SW_Push, U1 RP2040, U2 MCP1700x-330xxTT, U4 W25Q16JVUXIQ TR, Y1 12 MHz

Commit message: Add files via upload
Parts:
- removed J2, J3: Conn_01x02_Pin, Connector_Hirose:Hirose_DF13-02P-1.25DSA_1x02_P1.25mm_Vertical, symbol Connector:Conn_01x02_Pin
- removed J5, J6, J7: Conn_01x07_Pin, Connector_Hirose:Hirose_DF13-07P-1.25DSA_1x07_P1.25mm_Vertical, symbol Connector:Conn_01x07_Pin
- added J2, J3: Conn_01x08_Pin, Connector_Molex:Molex_SL_171971-0008_1x08_P2.54mm_Vertical, symbol Connector:Conn_01x08_Pin
Connections:
- net 3.3V: now also J3.8 (Pin_8)
- net GND: now also J2.8 (Pin_8)
- net GPIO0: now also J2.1 (Pin_1)
- net GPIO1: now also J2.2 (Pin_2)
- net GPIO18: now also J3.1 (Pin_1)
- net GPIO19: now also J3.2 (Pin_2)
- net GPIO2: now also J2.3 (Pin_3)
- net GPIO20: now also J3.3 (Pin_3)
- net GPIO21: now also J3.4 (Pin_4)
- net GPIO22: now also U1.25 (SWD), J3.7 (Pin_7)
- net GPIO23: now also J3.6 (Pin_6)
- net GPIO24: now also J3.5 (Pin_5)
- net GPIO3: now also J2.4 (Pin_4)
- net GPIO4: now also J2.5 (Pin_5)
- net GPIO5: now also J2.6 (Pin_6)
- net GPIO6: now also U1.24 (SWCLK), J2.7 (Pin_7)
- net GPIO10: no longer names the net of U1.13 (GPIO10)
- net GPIO11: no longer names the net of U1.14 (GPIO11)
- net GPIO12: no longer names the net of U1.15 (GPIO12)
- net GPIO13: no longer names the net of U1.16 (GPIO13)
- net GPIO14: no longer names the net of U1.17 (GPIO14)
- net GPIO14: no longer U1.25 (SWD)
- net GPIO8: no longer names the net of U1.11 (GPIO8)
- net GPIO8: no longer U1.24 (SWCLK)
- net GPIO9: no longer names the net of U1.12 (GPIO9)
- net RUN: no longer names the net of U1.26 (RUN)
- no-connect marks 5 -> 13
